Commit message: feat: add sim launch and foxglove bridge, refactor URDF mesh paths, and update Gazebo camera sensor configuration.

File: urdf/bcr_bot.xacro (robot description, xacro)
@@ -71,5 +71,5 @@
             <origin xyz="0 0 -0.205" rpy="0 0 0" />
             <geometry>
-                <mesh filename="file://$(find bcr_bot)/meshes/bcr_bot_mesh.dae" scale="1 1 1"/>
+                <mesh filename="package://bcr_bot/meshes/bcr_bot_mesh.dae" scale="1 1 1"/>
             </geometry>
         </visual>
@@ -142,5 +142,5 @@
                 <origin xyz="0 0 0" rpy="0 0 0" />
                 <geometry>
-                    <mesh filename="file://$(find bcr_bot)/meshes/kinect/d415.dae"/>
+                    <mesh filename="package://bcr_bot/meshes/kinect/d415.dae"/>
                 </geometry>
                 <material name="black"/>
@@ -176,5 +176,5 @@
                 <origin xyz="0 0 0" rpy="0 0 0" />
                 <geometry>
-                    <mesh filename="file://$(find bcr_bot)/meshes/kinect/d415.dae"/>
+                    <mesh filename="package://bcr_bot/meshes/kinect/d415.dae"/>
                 </geometry>
                 <material name="black"/>

File: urdf/gz.xacro (robot description, xacro)
@@ -9,4 +9,6 @@
         </plugin>
         <plugin filename="gz-sim-joint-state-publisher-system" name="gz::sim::systems::JointStatePublisher">
+            <joint_name>middle_left_wheel_joint</joint_name>
+            <joint_name>middle_right_wheel_joint</joint_name>
         </plugin>
         <!-- ........................... DIFFERENTIAL DRIVE PLUGIN ................................... -->
@@ -75,10 +77,29 @@
     <xacro:if value="$(arg camera_enabled)">
         <gazebo reference="kinect_camera">
-            <sensor type="depth_camera" name="kinect_camera">
+            <!-- RGB Camera for Image and CameraInfo (Uses optical frame for Foxglove Z-forward projection) -->
+            <sensor type="camera" name="kinect_camera">
+                <update_rate>30.0</update_rate>
+                <topic>kinect_camera/image</topic>
+                <gz_frame_id>kinect_camera_optical</gz_frame_id>
+                <camera>
+                    <camera_info_topic>kinect_camera/camera_info</camera_info_topic>
+                    <horizontal_fov>${radians(camera_horizontal_fov)}</horizontal_fov>
+                    <image>
+                        <width>640</width>
+                        <height>480</height>
+                        <format>R8G8B8</format>
+                    </image>
+                    <clip>
+                        <near>0.05</near>
+                        <far>8.0</far>
+                    </clip>
+                </camera>
+            </sensor>
+            <!-- Depth Camera for PointCloud (Uses robot frame for X-forward points) -->
+            <sensor type="depth_camera" name="kinect_camera_depth">
                 <update_rate>30.0</update_rate>
                 <topic>kinect_camera</topic>
                 <gz_frame_id>kinect_camera</gz_frame_id>
                 <camera>
-                    <camera_info_topic>kinect_camera/camera_info</camera_info_topic>
                     <horizontal_fov>${radians(camera_horizontal_fov)}</horizontal_fov>
                     <image>

Commit message: added changes to support multi robot sim

File: urdf/bcr_bot.xacro (robot description, xacro)
@@ -39,6 +39,4 @@
     <xacro:arg name="sim_ign" default="false" />
     <xacro:arg name="sim_gz" default="false" />
-    <xacro:arg name="odometry_source" default="world" />
-    <xacro:property name="odometry_source" value="$(arg odometry_source)"/>
     <!-- ............................... LOAD MACROS ................................. -->
     <xacro:include filename="$(find bcr_bot)/urdf/materials.xacro"/>

File: urdf/gz.xacro (robot description, xacro)
@@ -1,11 +1,8 @@
 <?xml version="1.0"?>
 <robot xmlns:xacro="http://www.ros.org/wiki/xacro" name="bcr_bot">
+    <xacro:property name="ns" value="$(arg robot_namespace)" scope="global"/>
+    <xacro:property name="tf_prefix_" value="${ns + '/' if ns != '' else ''}" scope="global"/>
     <!-- ........................... SENSOR PLUGIN ................................... -->
     <gazebo>
-        <plugin filename="gz-sim-sensors-system" name="gz::sim::systems::Sensors">
-            <render_engine>ogre2</render_engine>
-        </plugin>
-        <plugin filename="gz-sim-imu-system" name="gz::sim::systems::Imu">
-        </plugin>
         <plugin filename="gz-sim-joint-state-publisher-system" name="gz::sim::systems::JointStatePublisher">
             <joint_name>middle_left_wheel_joint</joint_name>
@@ -19,34 +16,18 @@
             <wheel_radius>${traction_wheel_radius+0.01}</wheel_radius>
             <odom_publish_frequency>30</odom_publish_frequency>
-            <topic>/cmd_vel</topic>
-            <xacro:if value="${odometry_source == 'encoders'}">
-                <odom_topic>$(arg wheel_odom_topic)</odom_topic>
-                <tf_topic>/tf</tf_topic>
-            </xacro:if>
-            <frame_id>odom</frame_id>
-            <child_frame_id>base_footprint</child_frame_id>
+            <topic>/$(arg robot_namespace)/cmd_vel</topic>
+            <odom_topic>$(arg wheel_odom_topic)</odom_topic>
+            <tf_topic>/tf</tf_topic>
+            <frame_id>${tf_prefix_}odom</frame_id>
+            <child_frame_id>${tf_prefix_}base_footprint</child_frame_id>
         </plugin>
     </gazebo>
-    <!-- ............................. ground truth .................................... -->
-    <xacro:if value="${odometry_source == 'world'}">
-    <gazebo>
-        <plugin filename="libgz-sim-odometry-publisher-system"
-            name="gz::sim::systems::OdometryPublisher">
-            <odom_frame>odom</odom_frame>
-            <robot_base_frame>base_footprint</robot_base_frame>
-            <odom_topic>$(arg wheel_odom_topic)</odom_topic>
-            <tf_topic>/tf</tf_topic>
-            <dimensions>2</dimensions>
-            <odom_publish_frequency>10</odom_publish_frequency>
-        </plugin>
-    </gazebo>
-    </xacro:if>
     <!-- ........................... 2D LIDAR config ................................... -->
     <xacro:if value="$(arg two_d_lidar_enabled)">
         <gazebo reference="two_d_lidar">
             <sensor name='gpu_lidar' type='gpu_lidar'>
-                <topic>scan</topic>
+                <topic>/$(arg robot_namespace)/scan</topic>
                 <update_rate>${two_d_lidar_update_rate}</update_rate>
-                <gz_frame_id>two_d_lidar</gz_frame_id>
+                <gz_frame_id>${tf_prefix_}two_d_lidar</gz_frame_id>
                 <lidar>
                     <scan>
@@ -81,5 +62,5 @@
                 <update_rate>30.0</update_rate>
                 <topic>kinect_camera/image</topic>
-                <gz_frame_id>kinect_camera_optical</gz_frame_id>
+                <gz_frame_id>${tf_prefix_}kinect_camera_optical</gz_frame_id>
                 <camera>
                     <camera_info_topic>kinect_camera/camera_info</camera_info_topic>
@@ -99,6 +80,6 @@
             <sensor type="depth_camera" name="kinect_camera_depth">
                 <update_rate>30.0</update_rate>
-                <topic>kinect_camera</topic>
-                <gz_frame_id>kinect_camera</gz_frame_id>
+                <topic>/$(arg robot_namespace)/kinect_camera</topic>
+                <gz_frame_id>${tf_prefix_}kinect_camera</gz_frame_id>
                 <camera>
                     <horizontal_fov>${radians(camera_horizontal_fov)}</horizontal_fov>
@@ -121,7 +102,7 @@
             <always_on>1</always_on>
             <update_rate>1</update_rate>
-            <gz_frame_id>imu_frame</gz_frame_id>
+            <gz_frame_id>${tf_prefix_}imu_frame</gz_frame_id>
             <visualize>true</visualize>
-            <topic>imu</topic>
+            <topic>/$(arg robot_namespace)/imu</topic>
         </sensor>
     </gazebo>
@@ -132,5 +113,5 @@
                 <update_rate>10.0</update_rate>
                 <always_on>true</always_on>
-                <gz_frame_id>stereo_camera_optical</gz_frame_id>
+                <gz_frame_id>${tf_prefix_}stereo_camera_optical</gz_frame_id>
                 <pose>0 -0.12 0 0 0 0</pose>
                 <topic>stereo_camera/right/image_raw</topic>
@@ -151,5 +132,5 @@
                 <update_rate>10.0</update_rate>
                 <always_on>true</always_on>
-                <gz_frame_id>stereo_camera_optical</gz_frame_id>
+                <gz_frame_id>${tf_prefix_}stereo_camera_optical</gz_frame_id>
                 <camera_info_topic>stereo_camera/left/camera_info</camera_info_topic>
                 <pose>0 0 0 0 0 0</pose>
